File: Phidias-F072-pcb.kicad_sch (KiCad schematic)
At the start: 2 parts

Commit message: Keyboard Matrix Finished
Parts:
- added C?: 10uF, symbol Device:C_Small
- added C? (x2): 4.7uF, symbol Device:C_Small
- added C? (x5): 100nF, symbol Device:C_Small
- added C?: 10nF, symbol Device:C_Small
- added C?: 1uF, symbol Device:C_Small
- added D?: 1N4148WT, Diode_SMD:D_SOD-523, symbol Diode:1N4148WT
- added LED? (x3): LED, symbol acheronSymbols:LED
- added Q?: 2N7002, Package_TO_SOT_SMD:SOT-23, symbol Transistor_FET:2N7002
- added R?: 10k, symbol Device:R_Small
- added R? (x2): 330, symbol Device:R_Small
- added R?: 330k, symbol Device:R_Small
- added R?: 100, symbol Device:R_Small
- added R?: 1k, symbol Device:R_Small
- added R?: 1M, symbol Device:R_Small
- added SW?: SW_Push, symbol Switch:SW_Push
Connections:
- net +3V3: now also C?.1, C?.1, C?.1, C?.1, C?.1, C?.1, C?.1, C?.1, SW?.1
- net BOOT0: now also C?.1, R?.2, R?.2
- net GND: now also C?.2, C?.2, C?.2, C?.2, C?.2, C?.2, C?.2, C?.2, C?.2, C?.2, LED?.K, LED?.K, LED?.K, Q?.2 (S), R?.1, R?.1
- net NRST: now also C?.1, R?.2
- new net: Q?.1 (G), R?.2, R?.2
- new net: LED?.A, R?.1
- new net: D?.1 (K), R?.1
- new net: LED?.A, LED?.A, R?.1
- new net: Q?.3 (D), R?.1
- new net: D?.2 (A), R?.1, SW?.2
- new net CAPS_INDICATOR: R?.2
- new net NUML_INDICATOR: R?.2
Other:
- added sheet Matrix (untitled.kicad_sch)
- note added: "DECOUPLING CAPS"
- note added: "JST"
- note added: "KEYBOARD MATRIX"
- note added: "LED INDICATORS"
- note added: "RESET"
- note added: "VDD 3 * 100nF + 4.7uF"
- note added: "VDDA 10nF + 1uF"
- note added: "VDDIO2 100nF + 4.7uF"
- moved on the sheet: J?
