File: untitled.kicad_sch (KiCad schematic)
At the start: 144 parts

Commit message: pcb laying
Parts:
- added SW83: Win key 1u, acheron_MX:MX100, symbol acheronSymbols:MXSwitch
- added SW86: LALT 6U, acheron_MX:MX150, symbol acheronSymbols:MXSwitch
- SW1, SW10, SW11, SW12, SW13, SW14, SW16, SW17, SW18, SW19, SW2, SW20, SW21, SW23, SW24, SW25, SW26, SW27, SW28, SW29, SW3, SW30, SW31, SW32, SW33, SW34, SW37, SW38, SW39, SW4, SW40, SW44, SW45, SW46, SW47, SW48, SW49, SW5, SW50, SW51, SW52, SW53, SW54, SW55, SW57, SW58, SW59, SW6, SW60, SW63, SW64, SW65, SW66, SW67, SW68, SW69, SW7, SW70, SW71, SW72, SW73, SW75, SW76, SW77, SW78, SW8, SW9, SW92, SW93, SW94, SW95, SW97, SW98: renamed from SW?; footprint (none) -> acheron_MX:MX100
- SW15: renamed from SW?; footprint (none) -> acheron_MX:MX200
- SW22, SW35, SW81, SW84, SW90, SW91: renamed from SW?; footprint (none) -> acheron_MX:MX150
- SW36: renamed from SW?; footprint (none) -> acheron_MX:MX_ISOEnter
- SW41, SW79: renamed from SW?; footprint (none) -> acheron_MX:MX200VR
- SW42, SW61, SW80, SW82, SW85: renamed from SW?; footprint (none) -> acheron_MX:MX125
- SW43, SW74: renamed from SW?; footprint (none) -> acheron_MX:MX175
- SW56, SW62: renamed from SW?; footprint (none) -> acheron_MX:MX225
- SW87: renamed from SW?; footprint (none) -> acheron_MX:MX600R
- SW88: renamed from SW?; footprint (none) -> acheron_MX:MX625R
- SW89: renamed from SW?; footprint (none) -> acheron_MX:MX700R
- SW96: renamed from SW?; footprint (none) -> acheron_MX:MX200R
- gave numbers to parts that had none: 48
Connections:
- net LALT: now also SW83.1 (Col)
- net ROW9: now also SW83.2 (Row), SW86.2 (Row)
- net LALT (6u): now reaches D42.2 (A), SW85.1 (Col)
- net LALT (6u): now also SW86.1 (Col)
Other:
- note added: "Win 1u key"
