File: Phidias-F072-pcb-backups/Phidias-F072-pcb-2022-09-16_132252/Phidias-F072-pcb.kicad_pcb (KiCad board)
At the start: 2 copper layers, 390.5 x 97 mm, 176 parts, among them J1 Conn_01x04_Female, J2 Conn_01x04_Female, Q1 2N7002, SW1 ESC, SW10 9, SW11 0, SW12 -, SW13 =, SW14 \ (SB), SW15 Full Backspace, SW16 Delete (SB), SW17 Delete, SW18 NumLock, SW19 /, SW2 1, SW20 *, SW21 -, SW22 Tab, SW23 Q, SW24 W, SW25 E, SW26 R, SW27 T, SW28 Y, SW29 U, SW3 2, SW30 I, SW31 O, SW32 P, SW33 [, SW34 ], SW35 Backspace (SB), SW36 ISO, SW37 PgUp, SW38 7, SW39 8, SW4 3, SW40 9, SW41 +, SW42 Stepped Capslock, SW43 CPSLCK, SW44 A, SW45 S, SW46 D, SW47 F, SW48 G, SW49 H, SW5 4, SW50 J, SW51 K, SW52 L, SW53 ;, SW54 '', SW55 1u ISO #, SW56 Enter, SW57 PgDown, SW58 4, SW59 5, SW6 5, SW60 6, SW61 LShift, SW62 Full LShift, SW63 \ (ISO), SW64 Z, SW65 X, SW66 C, SW67 V, SW68 B, SW69 N, SW7 6, SW70 M, SW71 ,, SW72 ., SW73 /, SW74 RShift, SW75 Up Arrow, SW76 1, SW77 2, SW78 3, SW79 NumPad Enter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

Commit message: Pre silk
Connections:
- D10 pad 3: COL8 -> COL9
- D19 pad 3: COL9 -> COL8
- D20 pad 3: COL8 -> COL9
- D29 pad 3: COL9 -> COL8
- D30 pad 3: COL8 -> COL9
- D39 pad 3: COL9 -> COL8
- D40 pad 3: COL8 -> COL9
- D47 pad 3: COL9 -> COL8
- D48 pad 3: COL8 -> COL9
- D9 pad 3: COL9 -> COL8
- U2 pad 17: unconnected-(U2-Pad17) -> ROW3
- U2 pad 18: unconnected-(U2-Pad18) -> ROW2
- U2 pad 26: unconnected-(U2-Pad26) -> COL6
- U2 pad 27: unconnected-(U2-Pad27) -> COL7
- U2 pad 28: unconnected-(U2-Pad28) -> ROW7
- U2 pad 29: unconnected-(U2-Pad29) -> ROW5
- U2 pad 30: unconnected-(U2-Pad30) -> ROW4
- U2 pad 31: unconnected-(U2-Pad31) -> ROW6
- U2 pad 38: unconnected-(U2-Pad38) -> COL9
- U2 pad 40: unconnected-(U2-Pad40) -> COL8
- U2 pad 42: unconnected-(U2-Pad42) -> COL5
Routing:
- net ROW3: track 335.6 -> 598.0 mm, vias 0 -> 1
- net ROW4: track 358.7 -> 588.2 mm, vias 0 -> 2
- net ROW5: track 291.2 -> 515.4 mm, vias 0 -> 2
- net COL9: track 66.7 -> 283.6 mm
- net ROW2: track 366.0 -> 582.1 mm
- net unconnected-(U2-Pad17): track 211.4 -> 0.00 mm
- net ROW6: track 361.1 -> 572.1 mm, vias 0 -> 2
- net ROW7: track 358.6 -> 563.9 mm, vias 0 -> 2
- net NUML_INDICATOR: track 10.1 -> 215.0 mm, vias 0 -> 2
- net unconnected-(U2-Pad18): track 169.3 -> 0.00 mm
- net COL8: track 75.1 -> 237.8 mm, vias 0 -> 2
- net GND: track 413.4 -> 559.3 mm, vias 5 -> 8
- net COL7: track 77.8 -> 208.7 mm, vias 2 -> 4
- net COL6: track 89.0 -> 170.9 mm, vias 0 -> 4
- net COL5: track 86.5 -> 142.6 mm, vias 0 -> 2
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