File: Phidias-F072-pcb-backups/Phidias-F072-pcb-2022-09-16_132252/Phidias-F072-pcb.kicad_sch (KiCad schematic)
At the start: 30 parts, among them J1 Conn_01x04_Female, J2 Conn_01x04_Female, Q1 2N7002, U1 XC6206PxxxMR, U2 STM32F072-LQFP48

Commit message: Pre silk
Connections:
- net COL5: now also U2.42 (I2C1_SCL/PB6)
- net COL6: now also U2.26 (SPI2_SCK/I2S2_CK/I2C2_SCL/PB13)
- net COL7: now also U2.27 (SPI2_MISO/I2S2_MCK/I2C2_SDA/TIM15_CH1/PB14)
- net COL8: now also U2.40 (SPI1_MISO/I2S1_MCK/TIM3_CH1/PB4)
- net COL9: now also U2.38 (PA15)
- net ROW2: now also U2.18 (PB0/TIM3_CH3/ADC_IN8)
- net ROW3: now also U2.17 (PA7/TIM3_CH2/TIM14_CH1/ADC_IN7)
- net ROW4: now also U2.30 (TIM1_CH2/PA9)
- net ROW5: now also U2.29 (TIM1_CH1/PA8)
- net ROW6: now also U2.31 (TIM1_CH3/PA10)
- net ROW7: now also U2.28 (SPI2_MOSI/I2S2_SD/PB15)
- no-connect marks 0 -> 11
Changed lines of the file:
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@@
   (junction (at 183.388 120.142) (diameter 0) (color 0 0 0 0)
   )
-  (junction (at 243.84 31.242) (diameter 0) (color 0 0 0 0)
-  )
   (junction (at 205.74 27.178) (diameter 0) (color 0 0 0 0)
   )
@@
   (junction (at 200.406 42.418) (diameter 0) (color 0 0 0 0)
   )
+  (no_connect (at 99.314 115.57))
+  (no_connect (at 33.274 93.98))
+  (no_connect (at 99.314 27.94))
+  (no_connect (at 73.914 27.94))
+  (no_connect (at 61.214 27.94))
+  (no_connect (at 54.864 27.94))
+  (no_connect (at 33.274 43.18))
+  (no_connect (at 33.274 49.53))
+  (no_connect (at 33.274 55.88))
+  (no_connect (at 33.274 62.23))
+  (no_connect (at 33.274 68.58))
   (polyline (pts (xy 143.002 64.008) (xy 218.694 64.008))
     (stroke (width 1) (type solid) (color 0 0 0 0))
@@
     (stroke (width 0) (type default) (color 0 0 0 0))
   )
-  (wire (pts (xy 243.84 31.242) (xy 259.08 31.242))
+  (wire (pts (xy 239.522 31.242) (xy 259.08 31.242))
     (stroke (width 0) (type default) (color 0 0 0 0))
   )
@@
   )
   (wire (pts (xy 258.572 63.5) (xy 258.572 64.516))
-    (stroke (width 0) (type default) (color 0 0 0 0))
-  )
-  (wire (pts (xy 239.522 31.242) (xy 243.84 31.242))
     (stroke (width 0) (type default) (color 0 0 0 0))
   )
@@
     (effects (font (size 1.27 1.27)) (justify left bottom))
   )
-  (global_label "COL8" (shape input) (at 2.286 88.138 0) (fields_autoplaced)
-    (effects (font (size 1.27 1.27)) (justify left))
-    (property "Intersheet References" "${INTERSHEET_REFS}" (id 0) (at 9.5372 88.0586 0)
+  (global_label "COL8" (shape input) (at 92.964 27.94 90) (fields_autoplaced)
+    (effects (font (size 1.27 1.27)) (justify left))
+    (property "Intersheet References" "${INTERSHEET_REFS}" (id 0) (at 92.8846 20.6888 90)
       (effects (font (size 1.27 1.27)) (justify left) hide)
     )
@@
     )
   )
-  (global_label "ROW4" (shape input) (at -10.414 68.58 0) (fields_autoplaced)
-    (effects (font (size 1.27 1.27)) (justify left))
-    (property "Intersheet References" "${INTERSHEET_REFS}" (id 0) (at -2.7395 68.5006 0)
-      (effects (font (size 1.27 1.27)) (justify left) hide)
-    )
-  )
-  (global_label "ROW5" (shape input) (at -11.176 72.898 0) (fields_autoplaced)
-    (effects (font (size 1.27 1.27)) (justify left))
-    (property "Intersheet References" "${INTERSHEET_REFS}" (id 0) (at -3.5015 72.8186 0)
+  (global_label "ROW4" (shape input) (at 120.904 76.2 0) (fields_autoplaced)
+    (effects (font (size 1.27 1.27)) (justify left))
+    (property "Intersheet References" "${INTERSHEET_REFS}" (id 0) (at 128.5785 76.1206 0)
+      (effects (font (size 1.27 1.27)) (justify left) hide)
+    )
+  )
+  (global_label "ROW5" (shape input) (at 120.904 82.55 0) (fields_autoplaced)
+    (effects (font (size 1.27 1.27)) (justify left))
+    (property "Intersheet References" "${INTERSHEET_REFS}" (id 0) (at 128.5785 82.4706 0)
       (effects (font (size 1.27 1.27)) (justify left) hide)
     )
@@
     )
   )
-  (global_label "COL6" (shape input) (at 2.286 78.74 0) (fields_autoplaced)
-    (effects (font (size 1.27 1.27)) (justify left))
-    (property "Intersheet References" "${INTERSHEET_REFS}" (id 0) (at 9.5372 78.6606 0)
+  (global_label "COL6" (shape input) (at 120.904 101.6 0) (fields_autoplaced)
+    (effects (font (size 1.27 1.27)) (justify left))
+    (property "Intersheet References" "${INTERSHEET_REFS}" (id 0) (at 128.1552 101.5206 0)
       (effects (font (size 1.27 1.27)) (justify left) hide)
     )
@@
     )
   )
-  (global_label "COL9" (shape input) (at 2.032 92.456 0) (fields_autoplaced)
-    (effects (font (size 1.27 1.27)) (justify left))
-    (property "Intersheet References" "${INTERSHEET_REFS}" (id 0) (at 9.2832 92.3766 0)
+  (global_label "COL9" (shape input) (at 105.664 27.94 90) (fields_autoplaced)
+    (effects (font (size 1.27 1.27)) (justify left))
+    (property "Intersheet References" "${INTERSHEET_REFS}" (id 0) (at 105.5846 20.6888 90)
       (effects (font (size 1.27 1.27)) (justify left) hide)
     )
@@
     )
   )
-  (global_label "ROW2" (shape input) (at -26.67 96.774 270) (fields_autoplaced)
-    (effects (font (size 1.27 1.27)) (justify right))
-    (property "Intersheet References" "${INTERSHEET_REFS}" (id 0) (at -26.5906 104.4485 90)
+  (global_label "ROW2" (shape input) (at 73.914 115.57 270) (fields_autoplaced)
+    (effects (font (size 1.27 1.27)) (justify right))
+    (property "Intersheet References" "${INTERSHEET_REFS}" (id 0) (at 73.9934 123.2445 90)
       (effects (font (size 1.27 1.27)) (justify right) hide)
     )
@@
     )
   )
-  (global_label "COL7" (shape input) (at 1.524 82.55 0) (fields_autoplaced)
-    (effects (font (size 1.27 1.27)) (justify left))
-    (property "Intersheet References" "${INTERSHEET_REFS}" (id 0) (at 8.7752 82.4706 0)
+  (global_label "COL7" (shape input) (at 120.904 95.25 0) (fields_autoplaced)
+    (effects (font (size 1.27 1.27)) (justify left))
+    (property "Intersheet References" "${INTERSHEET_REFS}" (id 0) (at 128.1552 95.1706 0)
       (effects (font (size 1.27 1.27)) (justify left) hide)
     )
@@
     )
   )
-  (global_label "COL5" (shape input) (at 2.794 73.406 0) (fields_autoplaced)
-    (effects (font (size 1.27 1.27)) (justify left))
-    (property "Intersheet References" "${INTERSHEET_REFS}" (id 0) (at 10.0452 73.3266 0)
+  (global_label "COL5" (shape input) (at 80.264 27.94 90) (fields_autoplaced)
+    (effects (font (size 1.27 1.27)) (justify left))
+    (property "Intersheet References" "${INTERSHEET_REFS}" (id 0) (at 80.1846 20.6888 90)
       (effects (font (size 1.27 1.27)) (justify left) hide)
     )
@@
     )
   )
-  (global_label "ROW7" (shape input) (at -11.43 82.296 0) (fields_autoplaced)
-    (effects (font (size 1.27 1.27)) (justify left))
-    (property "Intersheet References" "${INTERSHEET_REFS}" (id 0) (at -3.7555 82.2166 0)
+  (global_label "ROW7" (shape input) (at 120.904 88.9 0) (fields_autoplaced)
+    (effects (font (size 1.27 1.27)) (justify left))
+    (property "Intersheet References" "${INTERSHEET_REFS}" (id 0) (at 128.5785 88.8206 0)
       (effects (font (size 1.27 1.27)) (justify left) hide)
     )
@@
     )
   )
-  (global_label "ROW6" (shape input) (at -11.43 77.724 0) (fields_autoplaced)
-    (effects (font (size 1.27 1.27)) (justify left))
-    (property "Intersheet References" "${INTERSHEET_REFS}" (id 0) (at -3.7555 77.6446 0)
+  (global_label "ROW6" (shape input) (at 120.904 69.85 0) (fields_autoplaced)
+    (effects (font (size 1.27 1.27)) (justify left))
+    (property "Intersheet References" "${INTERSHEET_REFS}" (id 0) (at 128.5785 69.7706 0)
       (effects (font (size 1.27 1.27)) (justify left) hide)
     )
@@
     )
   )
-  (global_label "ROW3" (shape input) (at -9.652 64.008 0) (fields_autoplaced)
-    (effects (font (size 1.27 1.27)) (justify left))
-    (property "Intersheet References" "${INTERSHEET_REFS}" (id 0) (at -1.9775 63.9286 0)
-      (effects (font (size 1.27 1.27)) (justify left) hide)
+  (global_label "ROW3" (shape input) (at 67.564 115.57 270) (fields_autoplaced)
+    (effects (font (size 1.27 1.27)) (justify right))
+    (property "Intersheet References" "${INTERSHEET_REFS}" (id 0) (at 67.6434 123.2445 90)
+      (effects (font (size 1.27 1.27)) (justify right) hide)
     )
   )
@@
     (pin "1")
     (pin "2")
-  )
-  (symbol (lib_id "power:VCC") (at 243.84 31.242 0) (unit 1)
-    (in_bom yes) (on_board yes) (fields_autoplaced)
-    (property "Reference" "#PWR04" (id 0) (at 243.84 35.052 0)
-      (effects (font (size 1.27 1.27)) hide)
-    )
-    (property "Value" "VCC" (id 1) (at 243.84 26.67 0))
-    (property "Footprint" "" (id 2) (at 243.84 31.242 0)
-      (effects (font (size 1.27 1.27)) hide)
-    )
-    (property "Datasheet" "" (id 3) (at 243.84 31.242 0)
-      (effects (font (size 1.27 1.27)) hide)
-    )
-    (pin "1")
   )
   (symbol (lib_id "acheronSymbols:LED") (at 265.43 121.666 0) (unit 1)
@@
       (reference "#PWR03") (unit 1) (value "+5V") (footprint "")
     )
-    (path "/32632833-6d18-419a-baf5-56a271b92c3a"
-      (reference "#PWR04") (unit 1) (value "VCC") (footprint "")
-    )
     (path "/b2fb9e77-6600-4496-90f1-134c4c6edb56"
