File: Phidias-F072-pcb-backups/Phidias-F072-pcb-2022-09-16_132252/untitled.kicad_sch (KiCad schematic)
At the start: 146 parts, among them SW1 ESC, SW10 9, SW11 0, SW12 -, SW13 =, SW14 \ (SB), SW15 Full Backspace, SW16 Delete (SB), SW17 Delete, SW18 NumLock, SW19 /, SW2 1, SW20 *, SW21 -, SW22 Tab, SW23 Q, SW24 W, SW25 E, SW26 R, SW27 T, SW28 Y, SW29 U, SW3 2, SW30 I, SW31 O, SW32 P, SW33 [, SW34 ], SW35 Backspace (SB), SW36 ISO, SW37 PgUp, SW38 7, SW39 8, SW4 3, SW40 9, SW41 +, SW42 Stepped Capslock, SW43 CPSLCK, SW44 A, SW45 S, SW46 D, SW47 F, SW48 G, SW49 H, SW5 4, SW50 J, SW51 K, SW52 L, SW53 ;, SW54 '', SW55 1u ISO #, SW56 Enter, SW57 PgDown, SW58 4, SW59 5, SW6 5, SW60 6, SW61 LShift, SW62 Full LShift, SW63 \ (ISO), SW64 Z, SW65 X, SW66 C, SW67 V, SW68 B, SW69 N, SW7 6, SW70 M, SW71 ,, SW72 ., SW73 /, SW74 RShift, SW75 Up Arrow, SW76 1, SW77 2, SW78 3, SW79 NumPad Enter, SW8 7, SW80 LCtrl 1.25, SW81 LCtrl 1.5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

Commit message: Pre silk
Connections:
- net COL8: now also D19.3 (K), D29.3 (K), D39.3 (K), D47.3 (K), D9.3 (K); no longer D10.3 (K), D20.3 (K), D30.3 (K), D40.3 (K), D48.3 (K)
- net COL9: now also D10.3 (K), D20.3 (K), D30.3 (K), D40.3 (K), D48.3 (K); no longer D19.3 (K), D29.3 (K), D39.3 (K), D47.3 (K), D9.3 (K)
Changed lines of the file:
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@@
     )
   )
-  (global_label "COL9" (shape input) (at 485.648 39.37 90) (fields_autoplaced)
+  (global_label "COL9" (shape input) (at 537.21 39.37 90) (fields_autoplaced)
     (effects (font (size 1.27 1.27) bold) (justify left))
-    (property "Intersheet References" "${INTERSHEET_REFS}" (id 0) (at 485.521 31.9284 90)
+    (property "Intersheet References" "${INTERSHEET_REFS}" (id 0) (at 537.083 31.9284 90)
       (effects (font (size 1.27 1.27) bold) (justify left) hide)
     )
@@
     )
   )
-  (global_label "COL8" (shape input) (at 537.21 39.37 90) (fields_autoplaced)
+  (global_label "COL8" (shape input) (at 485.648 39.37 90) (fields_autoplaced)
     (effects (font (size 1.27 1.27) bold) (justify left))
-    (property "Intersheet References" "${INTERSHEET_REFS}" (id 0) (at 537.083 31.9284 90)
+    (property "Intersheet References" "${INTERSHEET_REFS}" (id 0) (at 485.521 31.9284 90)
       (effects (font (size 1.27 1.27) bold) (justify left) hide)
     )
